File: Front-End/Lochraster_Prototyp1/Oszi_Prototyp1/Oszi_Prototyp1.kicad_pcb (KiCad board)
At the start: 2 copper layers, 54.6 x 23.5 mm, 10 parts, among them IC1 LTC1420CGN#PBF, J1 FPGA_GPIO, J2 input

Commit message: 18.03.202123:41:19,54
Parts:
- removed REF**: 0Ohm, Resistor_SMD:R_1206_3216Metric_Pad1.42x1.75mm_HandSolder
Connections:
- C3 pad 1: +5V -> Net-(C3-Pad1)
- IC1 pad 3: +5V -> Net-(C3-Pad1)
Routing:
- net +5V: track 45.3 -> 36.0 mm
- net Net-(C3-Pad1): track 0.00 -> 5.98 mm
Changed lines of the file:
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@@
     (thickness 1.6)
     (drawings 9)
-    (tracks 185)
+    (tracks 181)
     (zones 0)
-    (modules 10)
-    (nets 43)
+    (modules 9)
+    (nets 44)
   )
   (page A4)
@@
   (net 41 "Net-(J1-Pad40)")
   (net 42 "Net-(J2-Pad2)")
+  (net 43 "Net-(C3-Pad1)")
   (net_class Default "Dies ist die voreingestellte Netzklasse."
     (clearance 0.25)
@@
     (add_net D9)
     (add_net GND)
+    (add_net "Net-(C3-Pad1)")
     (add_net "Net-(C5-Pad1)")
     (add_net "Net-(IC1-Pad1)")
@@
     (add_net OF)
   )
-  (module Resistor_SMD:R_1206_3216Metric_Pad1.42x1.75mm_HandSolder (layer F.Cu)
-    (at 130.175 57.15 90)
-    (descr "Resistor SMD 1206 (3216 Metric), square (rectangular) end terminal, IPC_7351 nominal with elongated pad for handsoldering. (Body size source: http://www.tortai-tech.com/upload/download/2011102023233369053.pdf), generated with kicad-footprint-generator")
-    (tags "resistor handsolder")
-    (attr smd)
-    (fp_text reference REF** (at 0 -1.82 90) (layer F.SilkS)
-      (effects (font (size 1 1) (thickness 0.15)))
-    )
-    (fp_text value 0Ohm (at 0.15 -1.925 90) (layer F.Fab)
-      (effects (font (size 1 1) (thickness 0.15)))
-    )
-    (fp_text user %R (at 0 0 90) (layer F.Fab)
-      (effects (font (size 0.8 0.8) (thickness 0.12)))
-    )
-    (fp_line (start 2.45 1.12) (end -2.45 1.12) (layer F.CrtYd) (width 0.05))
-    (fp_line (start 2.45 -1.12) (end 2.45 1.12) (layer F.CrtYd) (width 0.05))
-    (fp_line (start -2.45 -1.12) (end 2.45 -1.12) (layer F.CrtYd) (width 0.05))
-    (fp_line (start -2.45 1.12) (end -2.45 -1.12) (layer F.CrtYd) (width 0.05))
-    (fp_line (start -0.602064 0.91) (end 0.602064 0.91) (layer F.SilkS) (width 0.12))
-    (fp_line (start -0.602064 -0.91) (end 0.602064 -0.91) (layer F.SilkS) (width 0.12))
-    (fp_line (start 1.6 0.8) (end -1.6 0.8) (layer F.Fab) (width 0.1))
-    (fp_line (start 1.6 -0.8) (end 1.6 0.8) (layer F.Fab) (width 0.1))
-    (fp_line (start -1.6 -0.8) (end 1.6 -0.8) (layer F.Fab) (width 0.1))
-    (fp_line (start -1.6 0.8) (end -1.6 -0.8) (layer F.Fab) (width 0.1))
-    (pad 2 smd roundrect (at 1.4875 0 90) (size 1.425 1.75) (layers F.Cu F.Paste F.Mask) (roundrect_rratio 0.175)
-      (net 2 GND))
-    (pad 1 smd roundrect (at -1.4875 0 90) (size 1.425 1.75) (layers F.Cu F.Paste F.Mask) (roundrect_rratio 0.175)
-      (net 2 GND))
-    (model ${KISYS3DMOD}/Resistor_SMD.3dshapes/R_1206_3216Metric.wrl
-      (at (xyz 0 0 0))
-      (scale (xyz 1 1 1))
-      (rotate (xyz 0 0 0))
-    )
-  )
   (module Capacitor_SMD:C_1206_3216Metric_Pad1.42x1.75mm_HandSolder (layer F.Cu)
     (at 155.575 57.15)
@@
       (net 2 GND))
     (pad 1 smd roundrect (at -1.4875 0) (size 1.425 1.75) (layers F.Cu F.Paste F.Mask) (roundrect_rratio 0.175439)
-      (net 1 +5V))
+      (net 43 "Net-(C3-Pad1)"))
     (model ${KISYS3DMOD}/Capacitor_SMD.3dshapes/C_1206_3216Metric.wrl
       (at (xyz 0 0 0))
@@
       (net 2 GND))
     (pad 3 smd rect (at -2.712 -2.858 270) (size 0.435 1.526) (layers F.Cu F.Paste F.Mask)
-      (net 1 +5V))
+      (net 43 "Net-(C3-Pad1)"))
     (pad 4 smd rect (at -2.712 -2.222 270) (size 0.435 1.526) (layers F.Cu F.Paste F.Mask)
       (net 2 GND))
@@
   (segment (start 143.338 63.183) (end 145.097 63.183) (width 0.25) (layer F.Cu) (net 1))
   (segment (start 145.097 63.183) (end 146.05 62.23) (width 0.25) (layer F.Cu) (net 1))
-  (segment (start 146.367 61.913) (end 148.762 61.913) (width 0.25) (layer F.Cu) (net 1))
-  (segment (start 146.05 62.23) (end 146.367 61.913) (width 0.25) (layer F.Cu) (net 1))
   (segment (start 145.733 60.007) (end 146.05 59.69) (width 0.25) (layer F.Cu) (net 1))
   (segment (start 143.338 60.007) (end 145.733 60.007) (width 0.25) (layer F.Cu) (net 1))
@@
   (segment (start 145.733 60.007) (end 145.733 60.008) (width 0.25) (layer F.Cu) (net 1))
   (segment (start 146.05 59.69) (end 146.05 60.325) (width 0.4) (layer F.Cu) (net 1))
-  (segment (start 146.367 61.912) (end 146.05 61.595) (width 0.25) (layer F.Cu) (net 1))
-  (segment (start 146.367 61.913) (end 146.367 61.912) (width 0.25) (layer F.Cu) (net 1))
   (segment (start 146.05 60.325) (end 146.05 61.595) (width 0.4) (layer F.Cu) (net 1))
   (segment (start 146.05 61.595) (end 146.05 62.23) (width 0.4) (layer F.Cu) (net 1))
   (segment (start 151.8645 59.373) (end 154.0875 57.15) (width 0.25) (layer F.Cu) (net 1))
   (segment (start 148.762 59.373) (end 151.8645 59.373) (width 0.25) (layer F.Cu) (net 1))
-  (segment (start 152.5005 61.913) (end 148.762 61.913) (width 0.25) (layer F.Cu) (net 1))
-  (segment (start 154.0875 63.5) (end 152.5005 61.913) (width 0.25) (layer F.Cu) (net 1))
+  (segment (start 152.5005 61.913) (end 148.762 61.913) (width 0.25) (layer F.Cu) (net 43))
+  (segment (start 154.0875 63.5) (end 152.5005 61.913) (width 0.25) (layer F.Cu) (net 43))
   (segment (start 136.9425 62.865) (end 133.1325 59.055) (width 0.4) (layer F.Cu) (net 2))
   (segment (start 139.065 62.865) (end 136.9425 62.865) (width 0.4) (layer F.Cu) (net 2))

Commit message: 25.03.202112:23:24,69
Parts:
- added REF**: R_1206_3216Metric_Pad1.42x1.75mm_HandSolder, Resistor_SMD:R_1206_3216Metric_Pad1.42x1.75mm_HandSolder, F.Cu at (130.5, 57.2)
Changed lines of the file:
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@@
     (tracks 181)
     (zones 0)
-    (modules 9)
+    (modules 10)
     (nets 44)
   )
@@
     (add_net OF)
   )
+  (module Resistor_SMD:R_1206_3216Metric_Pad1.42x1.75mm_HandSolder (layer F.Cu)
+    (at 130.5 57.25 90)
+    (descr "Resistor SMD 1206 (3216 Metric), square (rectangular) end terminal, IPC_7351 nominal with elongated pad for handsoldering. (Body size source: http://www.tortai-tech.com/upload/download/2011102023233369053.pdf), generated with kicad-footprint-generator")
+    (tags "resistor handsolder")
+    (attr smd)
+    (fp_text reference REF** (at 0 -1.82 90) (layer F.SilkS)
+      (effects (font (size 1 1) (thickness 0.15)))
+    )
+    (fp_text value R_1206_3216Metric_Pad1.42x1.75mm_HandSolder (at 0 1.82 90) (layer F.Fab)
+      (effects (font (size 1 1) (thickness 0.15)))
+    )
+    (fp_text user %R (at 0 0 90) (layer F.Fab)
+      (effects (font (size 0.8 0.8) (thickness 0.12)))
+    )
+    (fp_line (start 2.45 1.12) (end -2.45 1.12) (layer F.CrtYd) (width 0.05))
+    (fp_line (start 2.45 -1.12) (end 2.45 1.12) (layer F.CrtYd) (width 0.05))
+    (fp_line (start -2.45 -1.12) (end 2.45 -1.12) (layer F.CrtYd) (width 0.05))
+    (fp_line (start -2.45 1.12) (end -2.45 -1.12) (layer F.CrtYd) (width 0.05))
+    (fp_line (start -0.602064 0.91) (end 0.602064 0.91) (layer F.SilkS) (width 0.12))
+    (fp_line (start -0.602064 -0.91) (end 0.602064 -0.91) (layer F.SilkS) (width 0.12))
+    (fp_line (start 1.6 0.8) (end -1.6 0.8) (layer F.Fab) (width 0.1))
+    (fp_line (start 1.6 -0.8) (end 1.6 0.8) (layer F.Fab) (width 0.1))
+    (fp_line (start -1.6 -0.8) (end 1.6 -0.8) (layer F.Fab) (width 0.1))
+    (fp_line (start -1.6 0.8) (end -1.6 -0.8) (layer F.Fab) (width 0.1))
+    (pad 2 smd roundrect (at 1.4875 0 90) (size 1.425 1.75) (layers F.Cu F.Paste F.Mask) (roundrect_rratio 0.175)
+      (net 2 GND))
+    (pad 1 smd roundrect (at -1.4875 0 90) (size 1.425 1.75) (layers F.Cu F.Paste F.Mask) (roundrect_rratio 0.175)
+      (net 2 GND))
+    (model ${KISYS3DMOD}/Resistor_SMD.3dshapes/R_1206_3216Metric.wrl
+      (at (xyz 0 0 0))
+      (scale (xyz 1 1 1))
+      (rotate (xyz 0 0 0))
+    )
+  )
   (module Capacitor_SMD:C_1206_3216Metric_Pad1.42x1.75mm_HandSolder (layer F.Cu)
     (at 155.575 57.15)
@@
   (segment (start 151.8645 59.373) (end 154.0875 57.15) (width 0.25) (layer F.Cu) (net 1))
   (segment (start 148.762 59.373) (end 151.8645 59.373) (width 0.25) (layer F.Cu) (net 1))
-  (segment (start 152.5005 61.913) (end 148.762 61.913) (width 0.25) (layer F.Cu) (net 43))
-  (segment (start 154.0875 63.5) (end 152.5005 61.913) (width 0.25) (layer F.Cu) (net 43))
   (segment (start 136.9425 62.865) (end 133.1325 59.055) (width 0.4) (layer F.Cu) (net 2))
   (segment (start 139.065 62.865) (end 136.9425 62.865) (width 0.4) (layer F.Cu) (net 2))
@@
   (segment (start 133.1325 55.88) (end 128.905 51.6525) (width 0.4) (layer F.Cu) (net 2))
   (segment (start 132.915 55.6625) (end 133.1325 55.88) (width 0.4) (layer F.Cu) (net 2))
+  (segment (start 132.715 58.6375) (end 133.1325 59.055) (width 0.4) (layer F.Cu) (net 2))
   (segment (start 130.175 55.6625) (end 132.915 55.6625) (width 0.4) (layer F.Cu) (net 2))
-  (segment (start 132.715 58.6375) (end 133.1325 59.055) (width 0.4) (layer F.Cu) (net 2))
   (segment (start 130.175 58.6375) (end 132.715 58.6375) (width 0.4) (layer F.Cu) (net 2))
   (segment (start 141.288 59.373) (end 143.338 59.373) (width 0.25) (layer F.Cu) (net 3))
@@
   (segment (start 139.7 66.04) (end 139.065 65.405) (width 0.4) (layer F.Cu) (net 42))
   (segment (start 144.78 66.04) (end 139.7 66.04) (width 0.4) (layer F.Cu) (net 42))
+  (segment (start 152.5005 61.913) (end 148.762 61.913) (width 0.25) (layer F.Cu) (net 43))
+  (segment (start 154.0875 63.5) (end 152.5005 61.913) (width 0.25) (layer F.Cu) (net 43))
   (zone (net 2) (net_name GND) (layer F.Cu) (hatch edge 0.508)
     (connect_pads (clearance 0.3))
